Commit message: ROM: display the visual model with rom transparency

File: data/urdf/solo_trunk.urdf (robot description, URDF)
Before this commit: robot solo_trunk, 1 links, 0 joints
Links:
- link base_link: geometry collision mesh filename=package://solo-rbprm/meshes/solo_trunk.stl; visual mesh filename=package://solo-rbprm/meshes/solo_all_visual.dae
